File: Schematic_PCB/SmartMonitor.kicad_sch (KiCad schematic)
At the start: 12 parts, among them J1 Screw_Terminal_01x02, J2 MQ135, J3 DHT22, U1 ZC323000, U2 LM2596T-5, U3 ESP-01

Commit message: Before RTOS
Parts:
- removed BZ1: Buzzer, symbol Device:Buzzer
- removed D2: LED, symbol Device:LED
- added J4: HW-417c, symbol Connector:Conn_01x06_Socket
- added SW1: SW_DIP_x02, symbol Switch:SW_DIP_x02
- added U4: DM-OLED096-636, DM-OLED096-636:MODULE_DM-OLED096-636, symbol DM-OLED096-636:DM-OLED096-636
- U1: value ZC323000 -> STM32
Connections:
- net GND: now also U1.19 (G), U3.1 (GND), J4.1 (Pin_1), U4.1 (GND)
- net at J2.1 (Pin_1): now also J3.1 (Pin_1), U1.38 (5V), SW1.1, SW1.2
- net at J2.4 (Pin_4): now also U1.10 (A5)
- net at C3.1, L1.2, U2.4 (FB): now also SW1.3
- net at U1.15 (B10): now also U3.4 (RXD)
- net at U1.16 (B11): now also U3.8 (TXD)
- net at U1.18 (3.3): now also U3.3 (GPIO0), U3.5 (VCC), U3.6 (~{RST}), U3.7 (CH_PD), U4.2 (VCC_IN)
- net at U1.26 (A9): now also J4.5 (Pin_5)
- net at U1.27 (A10): now also J4.4 (Pin_4)
- net at U1.34 (B6): now also U4.3 (SCL)
- net at U1.35 (B7): now also U4.4 (SDA)
- net at U1.6 (A1): now also J3.2 (Pin_2)
- new net: J4.3 (Pin_3), SW1.4
Other:
- note added: "GND CTS VCC TX RX DTR"
- moved on the sheet: J2, J3, U1, U3
